Commit message: eviscarated the vito robot description - works in Rviz now

File: lwr_velvet_description/gazebo/gazebo.urdf.xacro (robot description, xacro)
@@ -3,5 +3,5 @@
   <gazebo>
     <plugin name="gazebo_ros_controller" filename="libgazebo_ros_control.so">
-      <robotNamespace>/apple</robotNamespace>
+      <robotNamespace>/lwr_velvet</robotNamespace>
     </plugin>
   </gazebo>

File: lwr_velvet_description/urdf/lwr_velvet.urdf.xacro (robot description, xacro)
@@ -1,37 +1,49 @@
 <?xml version="1.0"?>
-<robot name="apple" xmlns:xacro="http://www.ros.org/wiki/xacro">
-  <!-- Import Rviz colors -->
-  <xacro:include filename="$(find apple_description)/urdf/materials.xacro" />
-  <!--Include the KUKA LBR iiwa-->
-  <xacro:include filename="$(find lbr_iiwa_description)/urdf/lbr_iiwa.xacro"/>
-  <!--Include the Velvet Fingers gripper-->
-  <xacro:include filename="$(find velvet_fingers_description)/urdf/velvet_fingers.xacro"/>
-   <!--Include the CitiTruck-->
-  <xacro:include filename="$(find apple_description)/urdf/citi_truck.xacro"/>
-   <!--Include the half pallet-->
-  <xacro:include filename="$(find apple_description)/urdf/half_pallet.xacro"/>
- <!-- Gazebo plugins -->
-  <xacro:include filename="$(find apple_description)/gazebo/gazebo.urdf.xacro"/>
-  <!-- Fix to world just for testing -->
-  <link name="world"/>
-  <!-- citi truck-->
-  <xacro:citi_truck name="citi_truck" parent="world">
-    <origin xyz="0 0 0" rpy="0 0 0" />
-  </xacro:citi_truck>
-  <!-- half pallet on the citi truck-->
-  <xacro:half_pallet name="transport_pallet" parent="citi_truck_base">
-    <origin xyz="0.6 0 0.02" rpy="0 0 0" />
-  </xacro:half_pallet>
-  <!-- half pallet for loading -->
-  <xacro:half_pallet name="load_pallet" parent="citi_truck_base">
-    <origin xyz="1.1 -0.9 0.02" rpy="0 0 0" />
-  </xacro:half_pallet>
-  <!--lbr -->
-  <xacro:lbr_iiwa name="lbr_iiwa" hardware_interface="$(arg prefix)" parent="citi_truck_base">
-    <origin xyz="0.114 -0.265 0.595" rpy="0 ${PI / 2} ${-PI / 4}" />
-  </xacro:lbr_iiwa>
-  <!--velvet fingers gripper -->
-  <xacro:velvet_fingers name="velvet_fingers" hardware_interface="$(arg prefix)" parent="lbr_iiwa_link_7">
-    <origin xyz="0 0 0.065" rpy="0 ${-PI / 2} 0" />
-  </xacro:velvet_fingers>
+<robot xmlns:xacro="http://www.ros.org/wiki/xacro"
+       name="lwr_velvet">
+<!-- RTKG: adapted from the Vito robot description -->
+  <!-- MODELS -->
+  <xacro:include filename="$(find lwr_velvet_description)/urdf/torso.urdf.xacro"/>
+  <xacro:include filename="$(find lwr_velvet_description)/urdf/table.urdf.xacro"/>
+  <xacro:include filename="$(find lwr_velvet_description)/urdf/materials.urdf"/>
+  <xacro:include filename="$(find lwr_description)/model/kuka_lwr.urdf.xacro"/>
+  <link name="world" />
+  <!-- BODY -->
+  <xacro:model_table name="table"
+                    parent="world"
+                    length="0.725"
+                    width="1.05"
+                    height="0.910"
+                    plate_thickness="0.05">
+    <origin xyz="-0.495 0.55 0" rpy="0 0 0"/>
+  </xacro:model_table>
+  <!-- WORKBENCH -->
+  <xacro:model_table name="workbench"
+                    parent="world"
+                    length="0.725"
+                    width="1.05"
+                    height="0.960"
+                    plate_thickness="0.1">
+  <origin xyz="-1.25 0.55 0.07" rpy="0 0 0"/>
+  </xacro:model_table>
+  <!-- TORSO -->
+  <xacro:model_torso name="torso" parent="world">
+    <origin xyz="0 0 0"/>
+  </xacro:model_torso>
+  <!-- LEFT ARM -->
+  <xacro:kuka_lwr name="left_arm" parent="world">
+    <origin xyz="-0.165 -0.1085854 0.390" rpy="1.5707963267948966 0.5235987010713441 -0.5235990737060282"/>
+  </xacro:kuka_lwr>
+  <!-- LEFT SOFTHAND
+  <xacro:soft_hand parent="left_arm_7_link" name="left_hand" left="true" withAdaptiveTransmission="true" useMimicTag="$(arg use_mimic_tag)">
+    <origin xyz="0 0 0" rpy="0 0 0"/>
+  </xacro:soft_hand-->
+  <!-- RIGHT ARM -->
+  <xacro:kuka_lwr name="right_arm" parent="world">
+    <origin xyz="-0.165 0.10858 0.390" rpy="-1.5707963267948966 0.5235987010713441 0.5235990737060282"/>
+  </xacro:kuka_lwr>
+  <!-- RIGHT SOFTHAND
+  <xacro:soft_hand parent="right_arm_7_link" name="right_hand" left="false" withAdaptiveTransmission="true" useMimicTag="$(arg use_mimic_tag)">
+    <origin xyz="0 0 0" rpy="0 0 0"/>
+  </xacro:soft_hand-->
 </robot>

File: lwr_velvet_description/urdf/materials.xacro (robot description, xacro)
@@ -1,4 +1,4 @@
 <?xml version="1.0"?>
-<robot name="apple" xmlns:xacro="http://www.ros.org/wiki/xacro">
+<robot name="lwr_velvet" xmlns:xacro="http://www.ros.org/wiki/xacro">
   <material name="Black">
     <color rgba="0.0 0.0 0.0 1.0"/>

Commit message: HQP control should work now for the Pisa setup

File: lwr_velvet_description/gazebo/gazebo.urdf.xacro (robot description, xacro)
@@ -1,4 +1,4 @@
 <?xml version="1.0"?>
-<robot name="apple" xmlns:xacro="http://www.ros.org/wiki/xacro">
+<robot name="lwr_velvet" xmlns:xacro="http://www.ros.org/wiki/xacro">
   <gazebo>
     <plugin name="gazebo_ros_controller" filename="libgazebo_ros_control.so">

File: lwr_velvet_description/urdf/lwr_velvet.urdf.xacro (robot description, xacro)
@@ -9,4 +9,5 @@
   <xacro:include filename="$(find lwr_description)/urdf/lwr.xacro"/>
   <xacro:include filename="$(find velvet_fingers_description)/urdf/velvet_fingers.xacro"/>
+  <xacro:include filename="$(find lwr_velvet_description)/gazebo/gazebo.urdf.xacro"/>
   <link name="world" />
   <!-- BODY -->
@@ -17,5 +18,5 @@
                     height="0.910"
                     plate_thickness="0.05">
-    <origin xyz="-0.495 0.55 0" rpy="0 0 0"/>
+    <origin xyz="-0.495 0.55 0.91" rpy="0 0 0"/>
   </xacro:model_table>
   <!-- WORKBENCH -->
@@ -26,9 +27,9 @@
                     height="0.960"
                     plate_thickness="0.1">
-  <origin xyz="-1.25 0.55 0.07" rpy="0 0 0"/>
+  <origin xyz="-1.25 0.55 0.98" rpy="0 0 0"/>
   </xacro:model_table>
   <!-- TORSO -->
   <xacro:model_torso name="torso" parent="world">
-    <origin xyz="0 0 0"/>
+    <origin xyz="0 0 0.91"/>
   </xacro:model_torso>
   <!-- LEFT ARM
@@ -41,6 +42,6 @@
   </xacro:soft_hand-->
   <!-- RIGHT ARM -->
-  <xacro:lwr name="right_arm" hardware_interface="$(arg prefix)" parent="world">
-    <origin xyz="-0.165 0.10858 0.390" rpy="-1.5707963267948966 0.5235987010713441 0.5235990737060282"/>
+  <xacro:lwr name="lwr" hardware_interface="$(arg prefix)" parent="world">
+    <origin xyz="-0.165 0.10858 1.3" rpy="-1.5707963267948966 0.5235987010713441 0.5235990737060282"/>
   </xacro:lwr>
   <!-- RIGHT SOFTHAND
@@ -49,5 +50,5 @@
   </xacro:soft_hand-->
   <!--velvet fingers gripper-->
-  <xacro:velvet_fingers name="velvet_fingers" hardware_interface="$(arg prefix)" parent="right_arm_link_7">
+  <xacro:velvet_fingers name="velvet_fingers" hardware_interface="$(arg prefix)" parent="lwr_link_7">
     <origin xyz="0 0 0.065" rpy="0 ${-PI / 2} 0" />
   </xacro:velvet_fingers>

File: lwr_velvet_description/urdf/table.urdf.xacro (robot description, xacro)
@@ -38,5 +38,6 @@
     </link>
     <gazebo reference="${name}_link">
-        <!-- <static>true</static> -->
+       <static>true</static>
+ <turnGravityOff>true</turnGravityOff>
     </gazebo>
 </xacro:macro>
@@ -78,5 +79,6 @@
     </xacro:table_leg>
     <gazebo reference="${name}_plate_link">
-        <!-- <static>true</static> -->
+        <static>true</static>
+ <turnGravityOff>true</turnGravityOff>
     </gazebo>
 </xacro:macro>

File: lwr_velvet_description/urdf/torso.urdf.xacro (robot description, xacro)
@@ -36,5 +36,6 @@
   </link>
   <gazebo reference="${name}_link">
-    <!-- <static>true</static> -->
+   <static>true</static>
+ <turnGravityOff>true</turnGravityOff>
   </gazebo>
 </xacro:macro>
