Commit message: adapted to Pisa urdf

File: lwr_description/urdf/lwr.transmission.xacro (robot description, xacro)
@@ -2,70 +2,70 @@
 <robot name="lwr" xmlns:xacro="http://www.ros.org/wiki/xacro">
   <xacro:macro name="lwr_transmission" params="name hardware_interface">
-    <transmission name="${name}_tran_1">
+    <transmission name="${name}_0_trans">
       <type>transmission_interface/SimpleTransmission</type>
-      <joint name="${name}_joint_1">
+      <joint name="${name}_0_joint">
 	<hardwareInterface>${hardware_interface}</hardwareInterface>
       </joint>
-      <actuator name="${name}_motor_1">
+      <actuator name="${name}_0_motor">
 	<hardwareInterface>${hardware_interface}</hardwareInterface>
 	<mechanicalReduction>1</mechanicalReduction>
       </actuator>
     </transmission>
-    <transmission name="${name}_tran_2">
+    <transmission name="${name}_1_trans">
       <type>transmission_interface/SimpleTransmission</type>
-      <joint name="${name}_joint_2">
+      <joint name="${name}_1_joint">
 	<hardwareInterface>${hardware_interface}</hardwareInterface>
       </joint>
-      <actuator name="${name}_motor_2">
+      <actuator name="${name}_1_motor">
 	<hardwareInterface>${hardware_interface}</hardwareInterface>
 	<mechanicalReduction>1</mechanicalReduction>
       </actuator>
     </transmission>
-    <transmission name="${name}_tran_3">
+    <transmission name="${name}_2_trans">
       <type>transmission_interface/SimpleTransmission</type>
-      <joint name="${name}_joint_3">
+      <joint name="${name}_2_joint">
 	<hardwareInterface>${hardware_interface}</hardwareInterface>
       </joint>
-      <actuator name="${name}_motor_3">
+      <actuator name="${name}_2_motor">
 	<hardwareInterface>${hardware_interface}</hardwareInterface>
 	<mechanicalReduction>1</mechanicalReduction>
       </actuator>
     </transmission>
-    <transmission name="${name}_tran_4">
+    <transmission name="${name}_3_trans">
       <type>transmission_interface/SimpleTransmission</type>
-      <joint name="${name}_joint_4">
+      <joint name="${name}_3_joint">
 	<hardwareInterface>${hardware_interface}</hardwareInterface>
       </joint>
-      <actuator name="${name}_motor_4">
+      <actuator name="${name}_3_motor">
 	<hardwareInterface>${hardware_interface}</hardwareInterface>
 	<mechanicalReduction>1</mechanicalReduction>
       </actuator>
     </transmission>
-    <transmission name="${name}_tran_5">
+    <transmission name="${name}_4_trans">
       <type>transmission_interface/SimpleTransmission</type>
-      <joint name="${name}_joint_5">
+      <joint name="${name}_4_joint">
 	<hardwareInterface>${hardware_interface}</hardwareInterface>
       </joint>
-      <actuator name="${name}_motor_5">
+      <actuator name="${name}_4_motor">
 	<hardwareInterface>${hardware_interface}</hardwareInterface>
 	<mechanicalReduction>1</mechanicalReduction>
       </actuator>
     </transmission>
-    <transmission name="${name}_tran_6">
+    <transmission name="${name}_5_trans">
       <type>transmission_interface/SimpleTransmission</type>
-      <joint name="${name}_joint_6">
+      <joint name="${name}_5_joint">
 	<hardwareInterface>${hardware_interface}</hardwareInterface>
       </joint>
-      <actuator name="${name}_motor_6">
+      <actuator name="${name}_5_motor">
 	<hardwareInterface>${hardware_interface}</hardwareInterface>
 	<mechanicalReduction>1</mechanicalReduction>
       </actuator>
     </transmission>
-    <transmission name="${name}_tran_7">
+    <transmission name="${name}_6_trans">
       <type>transmission_interface/SimpleTransmission</type>
-      <joint name="${name}_joint_7">
+      <joint name="${name}_6_joint">
 	<hardwareInterface>${hardware_interface}</hardwareInterface>
       </joint>
-      <actuator name="${name}_motor_7">
+      <actuator name="${name}_6_motor">
 	<hardwareInterface>${hardware_interface}</hardwareInterface>
 	<mechanicalReduction>1</mechanicalReduction>

File: lwr_description/urdf/lwr.xacro (robot description, xacro)
@@ -9,8 +9,4 @@
   <!-- Include Materials -->
   <xacro:include filename="$(find lwr_description)/urdf/materials.xacro"/>
-  <!-- my constants
-       <xacro:property name="joint_damping" value="0.5" />
-       <xacro:property name="max_effort" value="300"/>
-       <xacro:property name="max_velocity" value="10"/-->
   <!-- properties /-->
   <xacro:property name="base_mass" value="2.0"/>
@@ -18,8 +14,8 @@
   <xacro:property name="velocity_scale" value="1"/>
   <xacro:property name="effort_scale" value="1"/>
-  <!-- reflex to stiffness
-       <xacro:property name="max_stiffness" value="5000"/>
-       <xacro:property name="min_stiffness" value="0"/>
-       <xacro:property name="rate_stiffness" value="20000"/-->
+  <!-- reflex to stiffness-->
+  <xacro:property name="max_stiffness" value="5000"/>
+  <xacro:property name="min_stiffness" value="0"/>
+  <xacro:property name="rate_stiffness" value="20000"/>
   <xacro:macro name="lwr" params="parent name hardware_interface *origin">
     <!--joint between {parent} and link_0-->
@@ -27,7 +23,7 @@
       <insert_block name="origin"/>
       <parent link="${parent}"/>
-      <child link="${name}_link_0"/>
-    </joint>
-    <link name="${name}_link_0">
+      <child link="${name}_0_link"/>
+    </joint>
+    <link name="${name}_0_link">
       <inertial>
 	<mass value="${base_mass}"/>
@@ -51,13 +47,21 @@
     </link>
     <!-- Second segment of the arm. Joint along z-axis -->
-    <joint name="${name}_joint_1" type="revolute">
+    <joint name="${name}_0_joint" type="revolute">
       <origin xyz="0 0 0.11" rpy="0 0 0"/>
       <axis xyz="0 0 1"/>
       <limit lower="${-170 * PI / 180}" upper="${170 * PI / 180}" effort="176" velocity="${velocity_scale * 110 * PI / 180}" />
       <dynamics friction="10.0" damping="1.0"/>
-      <parent link="${name}_link_0"/>
-      <child link="${name}_link_1"/>
-    </joint>
-    <link name="${name}_link_1">
+      <parent link="${name}_0_link"/>
+      <child link="${name}_1_link"/>
+    </joint>
+    <joint name="${name}_0_joint_stiffness" type="revolute">
+      <axis xyz="0 0 1"/>
+      <limit lower="${min_stiffness}" upper="${max_stiffness}" effort="0" velocity="${rate_stiffness}" />
+      <safety_controller soft_lower_limit="${min_stiffness}" soft_upper_limit="${max_stiffness}" k_position="30" k_velocity="30"/>
+      <parent link="${name}_0_link"/>
+      <child link="${name}_1_link_dummy"/>
+    </joint>
+    <link name="${name}_1_link_dummy"/>
+    <link name="${name}_1_link">
       <inertial>
 	<mass value="${link_mass}"/>
@@ -93,13 +97,21 @@
     </link>
     <!-- Third segment of the arm. Joint along y-axis -->
-    <joint name="${name}_joint_2" type="revolute">
+    <joint name="${name}_1_joint" type="revolute">
       <origin xyz="0 0 0.2005" rpy="0 0 0"/>
       <axis xyz="0 -1 0"/>
       <limit lower="${-120 * PI / 180}" upper="${120 * PI / 180}" effort="176" velocity="${velocity_scale * 110 * PI / 180}" />
       <dynamics friction="10.0" damping="1.0"/>
-      <parent link="${name}_link_1"/>
-      <child link="${name}_link_2"/>
-    </joint>
-    <link name="${name}_link_2">
+      <parent link="${name}_1_link"/>
+      <child link="${name}_2_link"/>
+    </joint>
+    <joint name="${name}_1_joint_stiffness" type="revolute">
+      <axis xyz="0 0 1"/>
+      <limit lower="${min_stiffness}" upper="${max_stiffness}" effort="0" velocity="${rate_stiffness}" />
+      <safety_controller soft_lower_limit="${min_stiffness}" soft_upper_limit="${max_stiffness}" k_position="30" k_velocity="30"/>
+      <parent link="${name}_1_link"/>
+      <child link="${name}_2_link_dummy"/>
+    </joint>
+    <link name="${name}_2_link_dummy"/>
+    <link name="${name}_2_link">
       <inertial>
 	<mass value="${link_mass}"/>
@@ -135,13 +147,21 @@
     </link>
     <!-- Fourth element of the arm. z-axis -->
-    <joint name="${name}_joint_3" type="revolute">
+    <joint name="${name}_2_joint" type="revolute">
       <origin xyz="0 0 0.20" rpy="0 0 0"/>
       <axis xyz="0 0 1"/>
       <limit lower="${-170 * PI / 180}" upper="${170 * PI / 180}" effort="100" velocity="${velocity_scale * 128 * PI / 180}" />
       <dynamics friction="10.0" damping="1.0"/>
-      <parent link="${name}_link_2"/>
-      <child link="${name}_link_3"/>
-    </joint>
-    <link name="${name}_link_3">
+      <parent link="${name}_2_link"/>
+      <child link="${name}_3_link"/>
+    </joint>
+    <joint name="${name}_2_joint_stiffness" type="revolute">
+      <axis xyz="0 0 1"/>
+      <limit lower="${min_stiffness}" upper="${max_stiffness}" effort="0" velocity="${rate_stiffness}" />
+      <safety_controller soft_lower_limit="${min_stiffness}" soft_upper_limit="${max_stiffness}" k_position="30" k_velocity="30"/>
+      <parent link="${name}_2_link"/>
+      <child link="${name}_3_link_dummy"/>
+    </joint>
+    <link name="${name}_3_link_dummy"/>
+    <link name="${name}_3_link">
       <inertial>
 	<mass value="${link_mass}"/>
@@ -177,13 +197,21 @@
     </link>
     <!-- fifth element of the arm. x-axis -->
-    <joint name="${name}_joint_4" type="revolute">
+    <joint name="${name}_3_joint" type="revolute">
       <origin xyz="0 0 0.20" rpy="0 0 0"/>
       <axis xyz="0 1 0"/>
       <limit lower="${-120 * PI / 180}" upper="${120 * PI / 180}" effort="100" velocity="${velocity_scale * 128 * PI / 180}" />
       <dynamics friction="10.0" damping="1.0"/>
-      <parent link="${name}_link_3"/>
-      <child link="${name}_link_4"/>
-    </joint>
-    <link name="${name}_link_4">
+      <parent link="${name}_3_link"/>
+      <child link="${name}_4_link"/>
+    </joint>
+    <joint name="${name}_3_joint_stiffness" type="revolute">
+      <axis xyz="0 0 1"/>
+      <limit lower="${min_stiffness}" upper="${max_stiffness}" effort="0" velocity="${rate_stiffness}" />
+      <safety_controller soft_lower_limit="${min_stiffness}" soft_upper_limit="${max_stiffness}" k_position="30" k_velocity="30"/>
+      <parent link="${name}_3_link"/>
+      <child link="${name}_4_link_dummy"/>
+    </joint>
+    <link name="${name}_4_link_dummy"/>
+    <link name="${name}_4_link">
       <inertial>
 	<mass value="${link_mass}"/>
@@ -219,13 +247,21 @@
     </link>
     <!-- Sixth element of the arm. z-axis -->
-    <joint name="${name}_joint_5" type="revolute">
+    <joint name="${name}_4_joint" type="revolute">
       <origin xyz="0 0 0.20" rpy="0 0 0"/>
       <axis xyz="0 0 1"/>
       <limit lower="${-170 * PI / 180}" upper="${170 * PI / 180}" effort="100" velocity="${velocity_scale * 204 * PI / 180}" />
       <dynamics friction="10.0" damping="1.0"/>
-      <parent link="${name}_link_4"/>
-      <child link="${name}_link_5"/>
-    </joint>
-    <link name="${name}_link_5">
+      <parent link="${name}_4_link"/>
+      <child link="${name}_5_link"/>
+    </joint>
+    <joint name="${name}_4_joint_stiffness" type="revolute">
+      <axis xyz="0 0 1"/>
+      <limit lower="${min_stiffness}" upper="${max_stiffness}" effort="0" velocity="${rate_stiffness}" />
+      <safety_controller soft_lower_limit="${min_stiffness}" soft_upper_limit="${max_stiffness}" k_position="30" k_velocity="30"/>
+      <parent link="${name}_4_link"/>
+      <child link="${name}_5_link_dummy"/>
+    </joint>
+    <link name="${name}_5_link_dummy"/>
+    <link name="${name}_5_link">
       <inertial>
 	<mass value="${link_mass}"/>
@@ -261,13 +297,21 @@
     </link>
     <!-- Seventh element of the arm. z-axis -->
-    <joint name="${name}_joint_6" type="revolute">
+    <joint name="${name}_5_joint" type="revolute">
       <origin xyz="0 0 0.19" rpy="0 0 0"/>
       <axis xyz="0 -1 0"/>
       <limit lower="${-120 * PI / 180}" upper="${120 * PI / 180}" effort="38" velocity="${velocity_scale * 184 * PI / 180}" />
       <dynamics friction="10.0" damping="1.0"/>
-      <parent link="${name}_link_5"/>
-      <child link="${name}_link_6"/>
-    </joint>
-    <link name="${name}_link_6">
+      <parent link="${name}_5_link"/>
+      <child link="${name}_6_link"/>
+    </joint>
+    <joint name="${name}_5_joint_stiffness" type="revolute">
+      <axis xyz="0 0 1"/>
+      <limit lower="${min_stiffness}" upper="${max_stiffness}" effort="0" velocity="${rate_stiffness}" />
+      <safety_controller soft_lower_limit="${min_stiffness}" soft_upper_limit="${max_stiffness}" k_position="30" k_velocity="30"/>
+      <parent link="${name}_5_link"/>
+      <child link="${name}_6_link_dummy"/>
+    </joint>
+    <link name="${name}_6_link_dummy"/>
+    <link name="${name}_6_link">
       <inertial>
 	<mass value="0.2"/>
@@ -290,13 +334,21 @@
     </link>
     <!-- Eighth element of the arm. z-axis -->
-    <joint name="${name}_joint_7" type="revolute">
+    <joint name="${name}_6_joint" type="revolute">
       <origin xyz="0 0 0.078" rpy="0 0 0"/>
       <axis xyz="0 0 1"/>
       <limit lower="${-170 * PI / 180}" upper="${170 * PI / 180}" effort="38" velocity="${velocity_scale * 184 * PI / 180}" />
       <dynamics friction="10.0" damping="1.0"/>
-      <parent link="${name}_link_6"/>
-      <child link="${name}_link_7"/>
-    </joint>
-    <link name="${name}_link_7">
+      <parent link="${name}_6_link"/>
+      <child link="${name}_7_link"/>
+    </joint>
+    <joint name="${name}_6_joint_stiffness" type="revolute">
+      <axis xyz="0 0 1"/>
+      <limit lower="${min_stiffness}" upper="${max_stiffness}" effort="0" velocity="${rate_stiffness}" />
+      <safety_controller soft_lower_limit="${min_stiffness}" soft_upper_limit="${max_stiffness}" k_position="30" k_velocity="30"/>
+      <parent link="${name}_6_link"/>
+      <child link="${name}_7_link_dummy"/>
+    </joint>
+    <link name="${name}_7_link_dummy"/>
+    <link name="${name}_7_link">
       <inertial>
 	<mass value="0.2"/>

File: lwr_velvet_description/urdf/lwr_velvet.urdf.xacro (robot description, xacro)
@@ -50,5 +50,5 @@
   </xacro:soft_hand-->
   <!--velvet fingers gripper-->
-  <xacro:velvet_fingers name="velvet_fingers" hardware_interface="$(arg prefix)" parent="lwr_link_7">
+  <xacro:velvet_fingers name="velvet_fingers" hardware_interface="$(arg prefix)" parent="lwr_7_link">
     <origin xyz="0 0 0.02" rpy="0 ${-PI / 2} 0" />
   </xacro:velvet_fingers>
