Commit message: reworked the PISA stuff for the LWR4+ arm

File: lwr_velvet_description/urdf/lwr_velvet.urdf.xacro (robot description, xacro)
@@ -6,6 +6,7 @@
   <xacro:include filename="$(find lwr_velvet_description)/urdf/torso.urdf.xacro"/>
   <xacro:include filename="$(find lwr_velvet_description)/urdf/table.urdf.xacro"/>
-  <xacro:include filename="$(find lwr_velvet_description)/urdf/materials.urdf"/>
-  <xacro:include filename="$(find lwr_description)/model/kuka_lwr.urdf.xacro"/>
+  <xacro:include filename="$(find lwr_velvet_description)/urdf/materials.xacro"/>
+  <xacro:include filename="$(find lwr_description)/urdf/lwr.xacro"/>
+  <xacro:include filename="$(find velvet_fingers_description)/urdf/velvet_fingers.xacro"/>
   <link name="world" />
   <!-- BODY -->
@@ -31,8 +32,8 @@
     <origin xyz="0 0 0"/>
   </xacro:model_torso>
-  <!-- LEFT ARM -->
-  <xacro:kuka_lwr name="left_arm" parent="world">
+  <!-- LEFT ARM
+  <xacro:lwr name="left_arm" hardware_interface="$(arg prefix)" parent="world">
     <origin xyz="-0.165 -0.1085854 0.390" rpy="1.5707963267948966 0.5235987010713441 -0.5235990737060282"/>
-  </xacro:kuka_lwr>
+  </xacro:lwr-->
   <!-- LEFT SOFTHAND
   <xacro:soft_hand parent="left_arm_7_link" name="left_hand" left="true" withAdaptiveTransmission="true" useMimicTag="$(arg use_mimic_tag)">
@@ -40,10 +41,14 @@
   </xacro:soft_hand-->
   <!-- RIGHT ARM -->
-  <xacro:kuka_lwr name="right_arm" parent="world">
+  <xacro:lwr name="right_arm" hardware_interface="$(arg prefix)" parent="world">
     <origin xyz="-0.165 0.10858 0.390" rpy="-1.5707963267948966 0.5235987010713441 0.5235990737060282"/>
-  </xacro:kuka_lwr>
+  </xacro:lwr>
   <!-- RIGHT SOFTHAND
   <xacro:soft_hand parent="right_arm_7_link" name="right_hand" left="false" withAdaptiveTransmission="true" useMimicTag="$(arg use_mimic_tag)">
     <origin xyz="0 0 0" rpy="0 0 0"/>
   </xacro:soft_hand-->
+  <!--velvet fingers gripper-->
+  <xacro:velvet_fingers name="velvet_fingers" hardware_interface="$(arg prefix)" parent="right_arm_link_7">
+    <origin xyz="0 0 0.065" rpy="0 ${-PI / 2} 0" />
+  </xacro:velvet_fingers>
 </robot>

File: lwr_velvet_description/urdf/materials.xacro (robot description, xacro)
@@ -1,32 +1,32 @@
 <?xml version="1.0"?>
 <robot name="lwr_velvet" xmlns:xacro="http://www.ros.org/wiki/xacro">
-  <material name="Black">
+  <material name="LWR_VELVET/Black">
     <color rgba="0.0 0.0 0.0 1.0"/>
   </material>
-  <material name="Blue">
+  <material name="LWR_VELVET/Blue">
     <color rgba="0.0 0.0 0.8 1.0"/>
   </material>
-  <material name="Green">
+  <material name="LWR_VELVET/Green">
     <color rgba="0.0 0.8 0.0 1.0"/>
   </material>
-  <material name="Grey">
+  <material name="LWR_VELVET/Grey">
     <color rgba="0.2 0.2 0.2 1.0"/>
   </material>
-  <material name="Orange">
+  <material name="LWR_VELVET/Orange">
     <color rgba="${255/255} ${108/255} ${10/255} 1.0"/>
   </material>
-  <material name="Brown">
+  <material name="LWR_VELVET/Brown">
     <color rgba="${222/255} ${207/255} ${195/255} 1.0"/>
   </material>
-  <material name="Red">
+  <material name="LWR_VELVET/Red">
     <color rgba="0.8 0.0 0.0 1.0"/>
   </material>
-  <material name="White">
+  <material name="LWR_VELVET/White">
     <color rgba="1.0 1.0 1.0 1.0"/>
   </material>
-  <material name="Aluminium">
+  <material name="LWR_VELVET/Aluminium">
     <color rgba="${118/255} ${115/255} ${111/255} 1.0"/>
   </material>
-  <material name="Wood">
+  <material name="LWR_VELVET/Wood">
     <color rgba="${128/255} ${70/255} ${27/255} 1.0"/>
   </material>

File: lwr_velvet_description/urdf/table.urdf.xacro (robot description, xacro)
@@ -29,5 +29,5 @@
 				<box size="${leg_width/2} -${leg_width} ${height - plate_thickness}"/>
 			</geometry>
-			<material name="Vito/Black"/>
+			<material name="LWR_VELVET/Grey"/>
 		</visual>
 		<collision>
@@ -56,5 +56,5 @@
                 <box size="${length} ${width} ${plate_thickness}"/>
 			</geometry>
-			<material name="Vito/LightGrey"/>
+			<material name="LWR_VELVET/White"/>
 		</visual>
         <collision>

File: lwr_velvet_description/urdf/torso.urdf.xacro (robot description, xacro)
@@ -25,11 +25,11 @@
     <visual>
       <geometry>
-        <mesh filename="package://vito_description/meshes/torso.stl"/>
+        <mesh filename="package://lwr_velvet_description/meshes/torso.stl"/>
       </geometry>
-      <material name="Vito/Silver"/>
+      <material name="LWR_VELVET/Aluminium"/>
     </visual>
     <collision>
       <geometry>
-        <mesh filename="package://vito_description/meshes/torso.stl"/>
+        <mesh filename="package://lwr_velvet_description/meshes/torso.stl"/>
       </geometry>
     </collision>

Commit message: gimme_beer works in Gazebo. Yay.

File: lwr_velvet_description/urdf/lwr_velvet.urdf.xacro (robot description, xacro)
@@ -51,5 +51,5 @@
   <!--velvet fingers gripper-->
   <xacro:velvet_fingers name="velvet_fingers" hardware_interface="$(arg prefix)" parent="lwr_link_7">
-    <origin xyz="0 0 0.065" rpy="0 ${-PI / 2} 0" />
+    <origin xyz="0 0 0.02" rpy="0 ${-PI / 2} 0" />
   </xacro:velvet_fingers>
 </robot>

Commit message: rviz with point clouds and the proper urdf

File: lwr_velvet_description/urdf/lwr_velvet.urdf.xacro (robot description, xacro)
@@ -50,5 +50,5 @@
   <!--velvet fingers gripper-->
   <xacro:velvet_fingers name="velvet_fingers" hardware_interface="$(arg prefix)" parent="lwr_7_link">
-    <origin xyz="0 0 0.02" rpy="0 ${-PI / 2} 0" />
+    <origin xyz="0 0 0.03" rpy="0 ${-PI / 2} 0" />
   </xacro:velvet_fingers>
 </robot>

Commit message: started adapting the aalto setup

File: lwr_velvet_description/urdf/lwr_velvet.urdf.xacro (robot description, xacro)
@@ -2,5 +2,5 @@
 <robot xmlns:xacro="http://www.ros.org/wiki/xacro"
        name="lwr_velvet">
-<!-- RTKG: adapted from the Vito robot description -->
+  <!-- RTKG: adapted from the Aalto robot description -->
   <!-- MODELS -->
   <xacro:include filename="$(find lwr_velvet_description)/urdf/torso.urdf.xacro"/>
@@ -9,43 +9,48 @@
   <xacro:include filename="$(find oru_lwr_description)/model/kuka_lwr.urdf.xacro"/>
   <xacro:include filename="$(find velvet_fingers_description)/urdf/velvet_fingers.xacro"/>
-  <link name="world" />
-  <!-- BODY -->
-  <xacro:model_table name="table"
-                    parent="world"
-                    length="0.725"
-                    width="1.05"
-                    height="0.910"
-                    plate_thickness="0.05">
-    <origin xyz="-0.495 0.55 0.91" rpy="0 0 0"/>
-  </xacro:model_table>
+  <link name="world">
+    <visual>
+      <origin xyz="0 0 0.0075" rpy="0 0 0"/>
+      <geometry>
+	<box size="2.0 3.0 0.015"/>
+      </geometry>
+    </visual>
+    <collision>
+      <origin xyz="0 0 0.0075" rpy="0 0 0"/>
+      <geometry>
+	<box size="2.0 0.1 0.015"/>
+      </geometry>
+    </collision>
+  </link>
+  <!-- TABLE -->
+  <!--xacro:model_table name="table"
+      parent="world"
+      length="0.725"
+      width="1.05"
+      height="0.910"
+      plate_thickness="0.05">
+      <origin xyz="-0.495 0.55 0.91" rpy="0 0 0"/>
+      </xacro:model_table-->
   <!-- WORKBENCH -->
-  <xacro:model_table name="workbench"
-                    parent="world"
-                    length="0.725"
-                    width="1.05"
-                    height="0.960"
-                    plate_thickness="0.1">
-  <origin xyz="-1.25 0.55 0.98" rpy="0 0 0"/>
-  </xacro:model_table>
+  <!--xacro:model_table name="workbench"
+      parent="world"
+      length="0.725"
+      width="1.05"
+      height="0.960"
+      plate_thickness="0.1">
+      <origin xyz="-1.25 0.55 0.98" rpy="0 0 0"/>
+      </xacro:model_table-->
   <!-- TORSO -->
-  <xacro:model_torso name="torso" parent="world">
-    <origin xyz="0 0 0.91"/>
-  </xacro:model_torso>
-  <!-- LEFT ARM
-  <xacro:lwr name="left_arm" hardware_interface="$(arg prefix)" parent="world">
-    <origin xyz="-0.165 -0.1085854 0.390" rpy="1.5707963267948966 0.5235987010713441 -0.5235990737060282"/>
-  </xacro:lwr-->
-  <!-- LEFT SOFTHAND
-  <xacro:soft_hand parent="left_arm_7_link" name="left_hand" left="true" withAdaptiveTransmission="true" useMimicTag="$(arg use_mimic_tag)">
-    <origin xyz="0 0 0" rpy="0 0 0"/>
-  </xacro:soft_hand-->
+  <!--xacro:model_torso name="torso" parent="world">
+      <origin xyz="0 0 0.91"/>
+      </xacro:model_torso-->
   <!-- RIGHT ARM -->
   <xacro:kuka_lwr name="lwr" parent="world" hardware_interface="$(arg prefix)">
-    <origin xyz="-0.165 0.10858 1.3" rpy="-1.5707963267948966 0.5235987010713441 0.5235990737060282"/>
+    <origin xyz="0 0 0.015" rpy="0 0 0"/>
   </xacro:kuka_lwr>
   <!-- RIGHT SOFTHAND
-  <xacro:soft_hand parent="right_arm_7_link" name="right_hand" left="false" withAdaptiveTransmission="true" useMimicTag="$(arg use_mimic_tag)">
-    <origin xyz="0 0 0" rpy="0 0 0"/>
-  </xacro:soft_hand-->
+       <xacro:soft_hand parent="right_arm_7_link" name="right_hand" left="false" withAdaptiveTransmission="true" useMimicTag="$(arg use_mimic_tag)">
+       <origin xyz="0 0 0" rpy="0 0 0"/>
+       </xacro:soft_hand-->
   <!--velvet fingers gripper-->
   <xacro:velvet_fingers name="velvet_fingers" hardware_interface="$(arg prefix)" parent="lwr_7_link">

Commit message: modified urdf to include the aalto spacers between wrist and flange plate

File: lwr_velvet_description/urdf/lwr_velvet.urdf.xacro (robot description, xacro)
@@ -55,5 +55,5 @@
   <!--velvet fingers gripper-->
   <xacro:velvet_fingers name="velvet_fingers" hardware_interface="$(arg prefix)" parent="lwr_7_link">
-    <origin xyz="0 0 0.03" rpy="0 ${-PI / 2} 0" />
+    <origin xyz="0 0 0.0265" rpy="0 ${-PI / 2} 0" />
   </xacro:velvet_fingers>
 </robot>
